File: pot_sensor.kicad_sch (KiCad schematic)
At the start: 50 parts, among them J1 USB_C_Receptacle_USB2.0_14P, SW1 EN, SW2 BOOT, U1 ESP32-C3, U2 BQ24074RGT, U3 TPS63900, U4 W25Q32JVSS, U5 USBLC6-2P6, U7 HDC3020DEFR, U8 TPS22917DBV, Y1 ABM8-40MHZ

Commit message: Save
Parts:
- D1: value LED -> RED; footprint LED_SMD:LED_Cree-XHP50_3V_HighDensity -> LED_SMD:LED_0603_1608Metric
- D2: value LED -> BLUE; footprint LED_SMD:LED_Cree-XHP50_3V_HighDensity -> LED_SMD:LED_0603_1608Metric
- J1: footprint Package_DFN_QFN:UQFN-16_1.8x2.6mm_P0.4mm -> Connector_USB:USB_C_Receptacle_GCT_USB4105-xx-A_16P_TopMnt_Horizontal
- R13, R14: footprint Package_SO:SOIC-8_3.9x4.9mm_P1.27mm -> Resistor_SMD:R_0402_1005Metric
Changed lines of the file:
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@@
 			)
 		)
-		(property "Value" "LED"
+		(property "Value" "BLUE"
 			(at 75.8825 53.34 0)
 			(show_name no)
@@
 			)
 		)
-		(property "Footprint" "LED_SMD:LED_Cree-XHP50_3V_HighDensity"
+		(property "Footprint" "LED_SMD:LED_0603_1608Metric"
 			(at 77.47 57.15 0)
 			(hide yes)
@@
 			)
 		)
-		(property "Footprint" "Package_SO:SOIC-8_3.9x4.9mm_P1.27mm"
+		(property "Footprint" "Resistor_SMD:R_0402_1005Metric"
 			(at 149.86 154.178 90)
 			(hide yes)
@@
 			)
 		)
-		(property "Footprint" "Package_SO:SOIC-8_3.9x4.9mm_P1.27mm"
+		(property "Footprint" "Resistor_SMD:R_0402_1005Metric"
 			(at 140.97 171.958 90)
 			(hide yes)
@@
 			)
 		)
-		(property "Value" "LED"
+		(property "Value" "RED"
 			(at 75.8825 63.5 0)
 			(show_name no)
@@
 			)
 		)
-		(property "Footprint" "LED_SMD:LED_Cree-XHP50_3V_HighDensity"
+		(property "Footprint" "LED_SMD:LED_0603_1608Metric"
 			(at 77.47 67.31 0)
 			(hide yes)
@@
 			)
 		)
-		(property "Footprint" "Package_DFN_QFN:UQFN-16_1.8x2.6mm_P0.4mm"
+		(property "Footprint" "Connector_USB:USB_C_Receptacle_GCT_USB4105-xx-A_16P_TopMnt_Horizontal"
 			(at 35.56 109.22 0)
 			(hide yes)

Commit message: Choosen references in mouser website
Parts:
- A1, C12, JSTconnector1: now left out of the parts list
- C1: PartNumber (none) -> GXT21BR71A475KE3L
- C10: PartNumber (none) -> GCQ0335C1H3R9CB1D
- C11: PartNumber (none) -> GRM0335C1H4R9BA1D
- C13, C14, C4: PartNumber (none) -> ZRB15XC80G106ME5D
- C15: footprint Capacitor_SMD:C_0201_0603Metric -> Capacitor_SMD:C_0402_1005Metric; PartNumber (none) -> GXT155C80J105KE1D
- C16, C17, C18, C7, C8, C9: PartNumber (none) -> KAF21BR71H104KM
- C2: PartNumber (none) -> KGM03BR50J105MH
- C3: PartNumber (none) -> MAASE32MSB7226MP
- C5, C6: PartNumber (none) -> 06031A300FAT2A
- D1: PartNumber (none) -> APT1608SURCK-AMT
- D2: PartNumber (none) -> APT1608VBC/D
- D3: PartNumber (none) -> BAT54WS-HE3_A-08
- J1: PartNumber (none) -> 640-USB4930-00-A
- L1: PartNumber (none) -> SRN4018BTA-2R2M
- L2: footprint Inductor_SMD:L_0201_0603Metric -> Inductor_SMD:L_01005_0402Metric; PartNumber (none) -> LQP02HV1N8B02L
- R1, R3: footprint Resistor_SMD:R_0402_1005Metric -> Resistor_SMD:R_1206_3216Metric; PartNumber (none) -> TNPW12061K00BXEA
- R10, R13, R4, R7: PartNumber (none) -> ESR01MZPF1002
- R11, R12: PartNumber (none) -> SR0805FR-474K7L
- R14: PartNumber (none) -> ESR01MZPF5103
- R2: PartNumber (none) -> RC0603FR-071K78L
- R5: PartNumber (none) -> RC0402FR-0736K5L
- R6: PartNumber (none) -> SR1206FR-7W22RL
- R8, R9: PartNumber (none) -> TNPW04025K10BEED
- SW1, SW2: PartNumber (none) -> PTS810SJK250SMTR
- U1: PartNumber (none) -> ESP32-C3
- U2: PartNumber (none) -> BQ24074RGTR
- U3: PartNumber (none) -> TPS63900DSKR
- U4: PartNumber (none) -> W25Q32JVSSIMTR
- U5: PartNumber (none) -> USBLC6-2P6
- U7: PartNumber (none) -> HDC3020DEFR
- U8: PartNumber (none) -> TPS22917DBVR
- Y1: PartNumber (none) -> ABM8-40-B2-T

Commit message: Updated powre distribution zones and added status LED
Parts:
- added D4: GREEN, LED_SMD:LED_0603_1608Metric, symbol Device:LED
- added R15: 60, Resistor_SMD:R_0201_0603Metric, symbol Device:R
Connections:
- net GND: now also D4.1 (K)
- net at U1.28 (U0TXD): now also R15.2
- new net: D4.2 (A), R15.1
- no-connect marks 14 -> 13

Commit message: Update to match JLCpcb part supplier part #
Parts:
- A1, C12, JSTconnector1: now not fitted
- C1: LCSC Part # (none) -> C2857993; PartNumber GXT21BR71A475KE3L -> (none)
- C10: LCSC Part # (none) -> C22374845; PartNumber GCQ0335C1H3R9CB1D -> (none)
- C11: LCSC Part # (none) -> C2180781; PartNumber GRM0335C1H4R9BA1D -> (none)
- C13, C14, C4: LCSC Part # (none) -> C76991; PartNumber ZRB15XC80G106ME5D -> (none)
- C15: footprint Capacitor_SMD:C_0402_1005Metric -> Capacitor_SMD:C_0201_0603Metric; LCSC Part # (none) -> C76930; PartNumber GXT155C80J105KE1D -> (none)
- C16, C17, C18, C7, C8, C9: LCSC Part # (none) -> C5137467; PartNumber KAF21BR71H104KM -> (none)
- C2: value 1µ -> 1u; LCSC Part # (none) -> C76930; PartNumber KGM03BR50J105MH -> (none)
- C3: LCSC Part # (none) -> C2918511; PartNumber MAASE32MSB7226MP -> (none)
- C5, C6: LCSC Part # (none) -> C113797; PartNumber 06031A300FAT2A -> (none)
- D1: LCSC Part # (none) -> C965799; PartNumber APT1608SURCK-AMT -> (none)
- D2: LCSC Part # (none) -> C965807; PartNumber APT1608VBC/D -> (none)
- D3: LCSC Part # (none) -> C5381403; PartNumber BAT54WS-HE3_A-08 -> (none)
- D4: LCSC Part # (none) -> C510026; PartNumber APT1608CGCK -> (none)
- J1: LCSC Part # (none) -> C2765186; PartNumber 640-USB4930-00-A -> (none)
- L1: footprint Inductor_SMD:L_Bourns-SRN4018 -> Inductor_SMD:L_1008_2520Metric; LCSC Part # (none) -> C42455362; PartNumber SRN4018BTA-2R2M -> (none)
- L2: LCSC Part # (none) -> C1333014; PartNumber LQP02HV1N8B02L -> (none)
- R1, R3: LCSC Part # (none) -> C2907440; PartNumber TNPW12061K00BXEA -> (none)
- R10, R13, R4, R7: LCSC Part # (none) -> C2906861; PartNumber ESR01MZPF1002 -> (none)
- R11, R12: LCSC Part # (none) -> C2907326; PartNumber SR0805FR-474K7L -> (none)
- R14: LCSC Part # (none) -> C2909365; PartNumber ESR01MZPF5103 -> (none)
- R15: value 60 -> 60R; LCSC Part # (none) -> C320980; PartNumber RK73H1HRTTCM60R4 -> (none)
- R2: LCSC Part # (none) -> C2974030; PartNumber RC0603FR-071K78L -> (none)
- R5: LCSC Part # (none) -> C42396638; PartNumber RC0402FR-0736K5L -> (none)
- R6: LCSC Part # (none) -> C25364; PartNumber SR1206FR-7W22RL -> (none)
- R8, R9: LCSC Part # (none) -> C2906948; PartNumber TNPW04025K10BEED -> (none)
- SW1, SW2: LCSC Part # (none) -> C221895; PartNumber PTS810SJK250SMTR -> (none)
- U1: LCSC Part # (none) -> C2838500; PartNumber ESP32-C3 -> (none)
- U2: LCSC Part # (none) -> C2861252; PartNumber BQ24074RGTR -> (none)
- U3: LCSC Part # (none) -> C1518762; PartNumber TPS63900DSKR -> (none)
- U4: LCSC Part # (none) -> C179173; PartNumber W25Q32JVSSIMTR -> (none)
- U5: LCSC Part # (none) -> C2827693; PartNumber USBLC6-2P6 -> (none)
- U7: LCSC Part # (none) -> C7472806; PartNumber HDC3020DEFR -> (none)
- U8: LCSC Part # (none) -> C2681320; PartNumber TPS22917DBVR -> (none)
- Y1: LCSC Part # (none) -> C1985459; PartNumber ABM8-40-B2-T -> (none)
Changed lines of the file:
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@@
 			)
 		)
-		(property "PartNumber" "KAF21BR71H104KM"
+		(property "LCSC Part #" "C5137467"
 			(at 260.35 87.63 0)
 			(hide yes)
@@
 			)
 		)
-		(property "PartNumber" "LQP02HV1N8B02L"
+		(property "LCSC Part #" "C1333014"
 			(at 222.25 67.31 90)
 			(hide yes)
@@
 			)
 		)
-		(property "PartNumber" "HDC3020DEFR "
+		(property "LCSC Part #" "C7472806"
 			(at 52.07 166.37 0)
 			(hide yes)
@@
 			)
 		)
-		(property "PartNumber" "06031A300FAT2A"
+		(property "LCSC Part #" "C113797"
 			(at 130.81 121.92 0)
 			(hide yes)
@@
 			)
 		)
-		(property "PartNumber" "GRM0335C1H4R9BA1D"
+		(property "LCSC Part #" "C2180781"
 			(at 214.63 71.12 0)
 			(hide yes)
@@
 			)
 		)
-		(property "PartNumber" "GCQ0335C1H3R9CB1D"
+		(property "LCSC Part #" "C22374845"
 			(at 229.87 71.12 0)
 			(hide yes)
@@
 			)
 		)
-		(property "PartNumber" "SR0805FR-474K7L"
+		(property "LCSC Part #" "C2907326"
 			(at 78.74 148.59 0)
 			(hide yes)
@@
 			)
 		)
-		(property "PartNumber" "06031A300FAT2A"
+		(property "LCSC Part #" "C113797"
 			(at 152.4 121.92 0)
 			(hide yes)
@@
 			)
 		)
-		(property "PartNumber" "RC0603FR-071K78L"
+		(property "LCSC Part #" "C2974030"
 			(at 35.56 59.69 90)
 			(hide yes)
@@
 			)
 		)
-		(property "PartNumber" "KAF21BR71H104KM"
+		(property "LCSC Part #" "C5137467"
 			(at 166.37 54.61 0)
 			(hide yes)
@@
 			)
 		)
-		(property "PartNumber" "TPS22917DBVR"
+		(property "LCSC Part #" "C2681320"
 			(at 123.19 86.36 0)
 			(hide yes)
@@
 			)
 		)
-		(property "PartNumber" "TNPW12061K00BXEA"
+		(property "LCSC Part #" "C2907440"
 			(at 85.09 67.31 90)
 			(hide yes)
@@
 			)
 		)
-		(property "PartNumber" "ZRB15XC80G106ME5D"
+		(property "LCSC Part #" "C76991"
 			(at 102.87 33.02 0)
 			(hide yes)
@@
 			)
 		)
-		(property "Footprint" "Inductor_SMD:L_Bourns-SRN4018"
+		(property "Footprint" "Inductor_SMD:L_1008_2520Metric"
 			(at 101.6 54.61 0)
 			(hide yes)
@@
 			)
 		)
-		(property "PartNumber" "SRN4018BTA-2R2M"
+		(property "LCSC Part #" "C42455362"
 			(at 101.6 54.61 0)
 			(hide yes)
@@
 			)
 		)
-		(property "PartNumber" "GXT21BR71A475KE3L"
+		(property "LCSC Part #" "C2857993"
 			(at 78.74 43.18 0)
 			(hide yes)
@@
 		(on_board yes)
 		(in_pos_files yes)
-		(dnp no)
+		(dnp yes)
 		(fields_autoplaced yes)
 		(property "Reference" "A1"
@@
 			)
 		)
-		(property "PartNumber" ""
-			(at 215.9 50.8 90)
-			(hide yes)
-			(show_name no)
-			(do_not_autoplace no)
-			(effects
-				(font
-					(size 1.27 1.27)
-				)
-			)
-		)
 		(pin "2"
 		)
@@
 			)
 		)
-		(property "PartNumber" "ABM8-40-B2-T"
+		(property "LCSC Part #" "C1985459"
 			(at 140.97 118.11 0)
 			(hide yes)
@@
 			)
 		)
-		(property "PartNumber" "BQ24074RGTR"
+		(property "LCSC Part #" "C2861252"
 			(at 54.61 49.53 0)
 			(hide yes)
@@
 			)
 		)
-		(property "PartNumber" "APT1608VBC/D"
+		(property "LCSC Part #" "C965807"
 			(at 77.47 57.15 0)
 			(hide yes)
@@
 			)
 		)
-		(property "PartNumber" "USBLC6-2P6 "
+		(property "LCSC Part #" "C2827693"
 			(at 73.66 99.06 0)
 			(hide yes)
@@
 			)
 		)
-		(property "Footprint" "Capacitor_SMD:C_0402_1005Metric"
+		(property "Footprint" "Capacitor_SMD:C_0201_0603Metric"
 			(at 137.16 164.1348 0)
 			(hide yes)
@@
 			)
 		)
-		(property "PartNumber" "GXT155C80J105KE1D"
+		(property "LCSC Part #" "C76930"
 			(at 133.35 165.1 90)
 			(hide yes)
@@
 			)
 		)
-		(property "PartNumber" "W25Q32JVSSIMTR "
+		(property "LCSC Part #" "C179173"
 			(at 229.87 127 0)
 			(hide yes)
@@
 		(on_board yes)
 		(in_pos_files yes)
-		(dnp no)
+		(dnp yes)
 		(property "Reference" "C12"
 			(at 102.87 154.3051 0)
@@
 			)
 		)
-		(property "PartNumber" ""
-			(at 114.3 160.02 0)
-			(hide yes)
-			(show_name no)
-			(do_not_autoplace no)
-			(effects
-				(font
-					(size 1.27 1.27)
-				)
-			)
-		)
 		(pin "2"
 		)
@@
 			)
 		)
-		(property "PartNumber" "ZRB15XC80G106ME5D"
+		(property "LCSC Part #" "C76991"
 			(at 204.47 64.77 0)
 			(hide yes)
@@
 			)
 		)
-		(property "PartNumber" "PTS810SJK250SMTR"
+		(property "LCSC Part #" "C221895"
 			(at 252.73 88.9 90)
 			(hide yes)
@@
 			)
 		)
-		(property "PartNumber" "KAF21BR71H104KM"
+		(property "LCSC Part #" "C5137467"
 			(at 273.05 137.16 0)
 			(hide yes)
@@
 			)
 		)
-		(property "PartNumber" "TNPW04025K10BEED"
+		(property "LCSC Part #" "C2906948"
 			(at 52.07 128.27 0)
 			(hide yes)
@@
 			)
 		)
-		(property "PartNumber" "TPS63900DSKR"
+		(property "LCSC Part #" "C1518762"
 			(at 115.57 49.53 0)
 			(hide yes)
@@
 			)
 		)
-		(property "PartNumber" "ESR01MZPF1002"
+		(property "LCSC Part #" "C2906861"
 			(at 260.35 78.74 0)
 			(hide yes)
@@
 			)
 		)
-		(property "PartNumber" "KAF21BR71H104KM"
+		(property "LCSC Part #" "C5137467"
 			(at 243.84 125.73 90)
 			(hide yes)
@@
 			)
 		)
-		(property "PartNumber" "ESP32-C3"
+		(property "LCSC Part #" "C2838500"
 			(at 186.69 99.06 0)
 			(hide yes)
@@
 			)
 		)
-		(property "PartNumber" "ESR01MZPF1002"
+		(property "LCSC Part #" "C2906861"
 			(at 149.86 152.4 90)
 			(hide yes)
@@
 			)
 		)
-		(property "PartNumber" "ESR01MZPF1002"
+		(property "LCSC Part #" "C2906861"
 			(at 40.64 69.85 90)
 			(hide yes)
@@
 			)
 		)
-		(property "PartNumber" "PTS810SJK250SMTR"
+		(property "LCSC Part #" "C221895"
 			(at 265.43 138.43 90)
 			(hide yes)
@@
 			)
 		)
-		(property "PartNumber" "SR0805FR-474K7L"
+		(property "LCSC Part #" "C2907326"
 			(at 69.85 147.32 0)
 			(hide yes)
@@
 			)
 		)
-		(property "PartNumber" "BAT54WS-HE3_A-08"
+		(property "LCSC Part #" "C5381403"
 			(at 144.78 156.21 90)
 			(hide yes)
@@
 			)
 		)
-		(property "PartNumber" "KAF21BR71H104KM"
+		(property "LCSC Part #" "C5137467"
 			(at 156.21 54.61 0)
 			(hide yes)
@@
 			)
 		)
-		(property "PartNumber" "ESR01MZPF5103"
+		(property "LCSC Part #" "C2909365"
 			(at 140.97 170.18 90)
 			(hide yes)
@@
 			)
 		)
-		(property "PartNumber" "RC0402FR-0736K5L"
+		(property "LCSC Part #" "C42396638"
 			(at 129.54 49.53 90)
 			(hide yes)
@@
 			)
 		)
-		(property "PartNumber" "MAASE32MSB7226MP"
+		(property "LCSC Part #" "C2918511"
 			(at 127 33.02 0)
 			(hide yes)
@@
 			)
 		)
-		(property "PartNumber" "APT1608SURCK-AMT"
+		(property "LCSC Part #" "C965799"
 			(at 77.47 67.31 0)
 			(hide yes)
@@
 			)
 		)
-		(property "PartNumber" "KAF21BR71H104KM"
+		(property "LCSC Part #" "C5137467"
 			(at 161.29 63.5 0)
 			(hide yes)
@@
 			)
 		)
-		(property "PartNumber" "TNPW04025K10BEED"
+		(property "LCSC Part #" "C2906948"
 			(at 55.88 128.27 0)
 			(hide yes)
@@
 			)
 		)
-		(property "PartNumber" "TNPW12061K00BXEA"
+		(property "LCSC Part #" "C2907440"
 			(at 85.09 57.15 90)
 			(hide yes)
@@
 			)
 		)
-		(property "PartNumber" "ESR01MZPF1002"
+		(property "LCSC Part #" "C2906861"
 			(at 273.05 128.27 0)
 			(hide yes)
@@
 			)
 		)
-		(property "PartNumber" "ZRB15XC80G106ME5D"
+		(property "LCSC Part #" "C76991"
 			(at 151.13 63.5 0)
 			(hide yes)
@@
 		(on_board yes)
 		(in_pos_files yes)
-		(dnp no)
+		(dnp yes)
 		(fields_autoplaced yes)
 		(property "Reference" "JSTconnector1"
@@
 			)
 		)
-		(property "PartNumber" ""
-			(at 30.48 15.24 90)
-			(hide yes)
-			(show_name no)
-			(do_not_autoplace no)
-			(effects
-				(font
-					(size 1.27 1.27)
-				)
-			)
-		)
 		(pin "-"
 		)
@@
 			)
 		)
-		(property "PartNumber" "SR1206FR-7W22RL"
+		(property "LCSC Part #" "C25364"
 			(at 160.02 118.11 90)
 			(hide yes)
@@
 			)
 		)
-		(property "Value" "1µ"
+		(property "Value" "1u"
 			(at 35.56 39.3699 0)
 			(show_name no)
@@
 			)
 		)
-		(property "PartNumber" "KGM03BR50J105MH"
+		(property "LCSC Part #" "C76930"
 			(at 31.75 38.1 0)
 			(hide yes)
@@
 			)
 		)
-		(property "PartNumber" "APT1608CGCK"
+		(property "LCSC Part #" "C510026"
 			(at 143.51 99.06 0)
 			(hide yes)
@@
 			)
 		)
-		(property "PartNumber" " 640-USB4930-00-A "
+		(property "LCSC Part #" "C2765186"
 			(at 31.75 109.22 0)
 			(hide yes)
@@
 			)
 		)
-		(property "Value" "60"
+		(property "Value" "60R"
 			(at 151.13 95.25 90)
 			(show_name no)
@@
 			)
 		)
-		(property "PartNumber" "RK73H1HRTTCM60R4"
+		(property "LCSC Part #" "C320980"
 			(at 151.13 99.06 90)
 			(hide yes)

Commit message: Updated PSRAM model to reduce prices pending PCB update
Parts:
- U4: value W25Q32JVSS -> W25Q80DVSNIG; footprint Package_SO:SOIC-8_5.3x5.3mm_P1.27mm -> Package_SO:SOIC-8_3.9x4.9mm_P1.27mm; LCSC Part # C179173 -> C401655
Changed lines of the file:
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@@
 			)
 		)
-		(property "Value" "W25Q32JVSS"
+		(property "Value" "W25Q80DVSNIG"
 			(at 231.394 115.824 0)
 			(show_name no)
@@
 			)
 		)
-		(property "Footprint" "Package_SO:SOIC-8_5.3x5.3mm_P1.27mm"
+		(property "Footprint" "Package_SO:SOIC-8_3.9x4.9mm_P1.27mm"
 			(at 229.87 127 0)
 			(hide yes)
@@
 			)
 		)
-		(property "LCSC Part #" "C179173"
+		(property "LCSC Part #" "C401655"
 			(at 229.87 127 0)
 			(hide yes)

Commit message: Updated schematic due to component changes
Parts:
- R6: footprint Resistor_SMD:R_1206_3216Metric -> Resistor_SMD:R_0201_0603Metric; LCSC Part # C25364 -> C7467268
Changed lines of the file:
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@@
 			)
 		)
-		(property "Footprint" "Resistor_SMD:R_1206_3216Metric"
+		(property "Footprint" "Resistor_SMD:R_0201_0603Metric"
 			(at 160.02 119.888 90)
 			(hide yes)
@@
 			)
 		)
-		(property "LCSC Part #" "C25364"
+		(property "LCSC Part #" "C7467268"
 			(at 160.02 118.11 90)
 			(hide yes)

Commit message: Pending another part re-selection
Parts:
- C10: footprint Capacitor_SMD:C_0201_0603Metric -> Capacitor_SMD:C_0402_1005Metric; LCSC Part # C22374845 -> C1566
- C11: footprint Capacitor_SMD:C_0201_0603Metric -> Capacitor_SMD:C_0402_1005Metric; LCSC Part # C2180781 -> C1855285
- C15, C2: footprint Capacitor_SMD:C_0201_0603Metric -> Capacitor_SMD:C_0402_1005Metric; LCSC Part # C76930 -> C77009
- L2: footprint Inductor_SMD:L_01005_0402Metric -> Inductor_SMD:L_0402_1005Metric; LCSC Part # C1333014 -> C77107
- R15: footprint Resistor_SMD:R_0201_0603Metric -> Resistor_SMD:R_0603_1608Metric; LCSC Part # C320980 -> C166918
- R6: footprint Resistor_SMD:R_0201_0603Metric -> Resistor_SMD:R_0402_1005Metric; LCSC Part # C7467268 -> C140177
Changed lines of the file:
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@@
 			)
 		)
-		(property "Footprint" "Inductor_SMD:L_01005_0402Metric"
+		(property "Footprint" "Inductor_SMD:L_0402_1005Metric"
 			(at 222.25 67.31 0)
 			(hide yes)
@@
 			)
 		)
-		(property "LCSC Part #" "C1333014"
+		(property "LCSC Part #" "C77107"
 			(at 222.25 67.31 90)
 			(hide yes)
@@
 			)
 		)
-		(property "Footprint" "Capacitor_SMD:C_0201_0603Metric"
+		(property "Footprint" "Capacitor_SMD:C_0402_1005Metric"
 			(at 215.5952 74.93 0)
 			(hide yes)
@@
 			)
 		)
-		(property "LCSC Part #" "C2180781"
+		(property "LCSC Part #" "C1855285"
 			(at 214.63 71.12 0)
 			(hide yes)
@@
 			)
 		)
-		(property "Footprint" "Capacitor_SMD:C_0201_0603Metric"
+		(property "Footprint" "Capacitor_SMD:C_0402_1005Metric"
 			(at 228.9048 67.31 0)
 			(hide yes)
@@
 			)
 		)
-		(property "LCSC Part #" "C22374845"
+		(property "LCSC Part #" "C1566"
 			(at 229.87 71.12 0)
 			(hide yes)
@@
 			)
 		)
-		(property "Footprint" "Capacitor_SMD:C_0201_0603Metric"
+		(property "Footprint" "Capacitor_SMD:C_0402_1005Metric"
 			(at 137.16 164.1348 0)
 			(hide yes)
@@
 			)
 		)
-		(property "LCSC Part #" "C76930"
+		(property "LCSC Part #" "C77009"
 			(at 133.35 165.1 90)
 			(hide yes)
@@
 			)
 		)
-		(property "Footprint" "Resistor_SMD:R_0201_0603Metric"
+		(property "Footprint" "Resistor_SMD:R_0402_1005Metric"
 			(at 160.02 119.888 90)
 			(hide yes)
@@
 			)
 		)
-		(property "LCSC Part #" "C7467268"
+		(property "LCSC Part #" "C140177"
 			(at 160.02 118.11 90)
 			(hide yes)
@@
 			)
 		)
-		(property "Footprint" "Capacitor_SMD:C_0201_0603Metric"
+		(property "Footprint" "Capacitor_SMD:C_0402_1005Metric"
 			(at 32.7152 41.91 0)
 			(hide yes)
@@
 			)
 		)
-		(property "LCSC Part #" "C76930"
+		(property "LCSC Part #" "C77009"
 			(at 31.75 38.1 0)
 			(hide yes)
@@
 			)
 		)
-		(property "Footprint" "Resistor_SMD:R_0201_0603Metric"
+		(property "Footprint" "Resistor_SMD:R_0603_1608Metric"
 			(at 151.13 100.838 90)
 			(hide yes)
@@
 			)
 		)
-		(property "LCSC Part #" "C320980"
+		(property "LCSC Part #" "C166918"
 			(at 151.13 99.06 90)
 			(hide yes)
