File: pot_sensor.kicad_sch (KiCad schematic)
At the start: 52 parts, among them J1 USB_C_Receptacle_USB2.0_14P, SW1 EN, SW2 BOOT, U1 ESP32-C3, U2 BQ24074RGT, U3 TPS63900, U4 W25Q80DVSNIG, U5 USBLC6-2P6, U7 HDC3020DEFR, U8 TPS22917DBV, Y1 ABM8-40MHZ

Commit message: New pieces
Parts:
- C1: footprint Capacitor_SMD:C_0805_2012Metric -> Capacitor_SMD:C_0402_1005Metric; LCSC Part # C2857993 -> C23733
- C10: LCSC Part # C1566 -> C1565
- C11: LCSC Part # C1855285 -> C1569
- C13, C14, C4: LCSC Part # C76991 -> C15525
- C15, C2: LCSC Part # C77009 -> C52923
- C16, C17, C18, C7, C8, C9: footprint Capacitor_SMD:C_0805_2012Metric -> Capacitor_SMD:C_0402_1005Metric; LCSC Part # C5137467 -> C1525
- C3: footprint Capacitor_SMD:C_1210_3225Metric -> Capacitor_SMD:C_0603_1608Metric; LCSC Part # C2918511 -> C59461
- C5, C6: footprint Capacitor_SMD:C_0603_1608Metric -> Capacitor_SMD:C_0402_1005Metric; LCSC Part # C113797 -> C1570
- D1: footprint LED_SMD:LED_0603_1608Metric -> LED_SMD:LED_0805_2012Metric; LCSC Part # C965799 -> C84256
- D2: value BLUE -> GREEN; footprint LED_SMD:LED_0603_1608Metric -> LED_SMD:LED_0805_2012Metric; LCSC Part # C965807 -> C2297
- D3: footprint Diode_SMD:D_SOD-323 -> Package_TO_SOT_SMD:SOT-23; LCSC Part # C5381403 -> C7502690
- D4: value GREEN -> YELLOW; LCSC Part # C510026 -> C89811
- L1: footprint Inductor_SMD:L_1008_2520Metric -> Inductor_SMD:L_0805_2012Metric; LCSC Part # C42455362 -> C1043
- R1, R3: footprint Resistor_SMD:R_1206_3216Metric -> Resistor_SMD:R_0402_1005Metric; LCSC Part # C2907440 -> C11702
- R10, R4, R7: footprint Resistor_SMD:R_0402_1005Metric -> Resistor_SMD:R_0603_1608Metric; LCSC Part # C2906861 -> C25804
- R11, R12: footprint Resistor_SMD:R_0805_2012Metric -> Resistor_SMD:R_0402_1005Metric; LCSC Part # C2907326 -> C25900
- R13: LCSC Part # C2906861 -> C25744
- R14: LCSC Part # C2909365 -> C11616
- R15: LCSC Part # C166918 -> C27592
- R2: LCSC Part # C2974030 -> C4177
- R5: footprint Resistor_SMD:R_0402_1005Metric -> Resistor_SMD:R_0603_1608Metric; LCSC Part # C42396638 -> C23147
- R6: LCSC Part # C140177 -> C25092
- R8, R9: LCSC Part # C2906948 -> C25905
- SW1, SW2: footprint Button_Switch_SMD:SW_SPST_PTS810 -> Button_Switch_SMD:SW_SPST_TS-1088-xR025; LCSC Part # C221895 -> C720477
Changed lines of the file:
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@@
 			)
 		)
-		(property "Footprint" "Capacitor_SMD:C_0805_2012Metric"
+		(property "Footprint" "Capacitor_SMD:C_0402_1005Metric"
 			(at 261.3152 91.44 0)
 			(hide yes)
@@
 			)
 		)
-		(property "LCSC Part #" "C5137467"
+		(property "LCSC Part #" "C1525"
 			(at 260.35 87.63 0)
 			(hide yes)
@@
 			)
 		)
-		(property "Footprint" "Capacitor_SMD:C_0603_1608Metric"
+		(property "Footprint" "Capacitor_SMD:C_0402_1005Metric"
 			(at 131.7752 125.73 0)
 			(hide yes)
@@
 			)
 		)
-		(property "LCSC Part #" "C113797"
+		(property "LCSC Part #" "C1570"
 			(at 130.81 121.92 0)
 			(hide yes)
@@
 			)
 		)
-		(property "LCSC Part #" "C1855285"
+		(property "LCSC Part #" "C1569"
 			(at 214.63 71.12 0)
 			(hide yes)
@@
 			)
 		)
-		(property "LCSC Part #" "C1566"
+		(property "LCSC Part #" "C1565"
 			(at 229.87 71.12 0)
 			(hide yes)
@@
 			)
 		)
-		(property "Footprint" "Resistor_SMD:R_0805_2012Metric"
+		(property "Footprint" "Resistor_SMD:R_0402_1005Metric"
 			(at 76.962 148.59 90)
 			(hide yes)
@@
 			)
 		)
-		(property "LCSC Part #" "C2907326"
+		(property "LCSC Part #" "C25900"
 			(at 78.74 148.59 0)
 			(hide yes)
@@
 			)
 		)
-		(property "Footprint" "Capacitor_SMD:C_0603_1608Metric"
+		(property "Footprint" "Capacitor_SMD:C_0402_1005Metric"
 			(at 153.3652 125.73 0)
 			(hide yes)
@@
 			)
 		)
-		(property "LCSC Part #" "C113797"
+		(property "LCSC Part #" "C1570"
 			(at 152.4 121.92 0)
 			(hide yes)
@@
 			)
 		)
-		(property "LCSC Part #" "C2974030"
+		(property "LCSC Part #" "C4177"
 			(at 35.56 59.69 90)
 			(hide yes)
@@
 			)
 		)
-		(property "Footprint" "Capacitor_SMD:C_0805_2012Metric"
+		(property "Footprint" "Capacitor_SMD:C_0402_1005Metric"
 			(at 167.3352 58.42 0)
 			(hide yes)
@@
 			)
 		)
-		(property "LCSC Part #" "C5137467"
+		(property "LCSC Part #" "C1525"
 			(at 166.37 54.61 0)
 			(hide yes)
@@
 			)
 		)
-		(property "Footprint" "Resistor_SMD:R_1206_3216Metric"
+		(property "Footprint" "Resistor_SMD:R_0402_1005Metric"
 			(at 85.09 69.088 90)
 			(show_name no)
@@
 			)
 		)
-		(property "LCSC Part #" "C2907440"
+		(property "LCSC Part #" "C11702"
 			(at 85.09 67.31 90)
 			(hide yes)
@@
 			)
 		)
-		(property "LCSC Part #" "C76991"
+		(property "LCSC Part #" "C15525"
 			(at 102.87 33.02 0)
 			(hide yes)
@@
 			)
 		)
-		(property "Footprint" "Inductor_SMD:L_1008_2520Metric"
+		(property "Footprint" "Inductor_SMD:L_0805_2012Metric"
 			(at 101.6 54.61 0)
 			(hide yes)
@@
 			)
 		)
-		(property "LCSC Part #" "C42455362"
+		(property "LCSC Part #" "C1043"
 			(at 101.6 54.61 0)
 			(hide yes)
@@
 			)
 		)
-		(property "Footprint" "Capacitor_SMD:C_0805_2012Metric"
+		(property "Footprint" "Capacitor_SMD:C_0402_1005Metric"
 			(at 79.7052 46.99 0)
 			(hide yes)
@@
 			)
 		)
-		(property "LCSC Part #" "C2857993"
+		(property "LCSC Part #" "C23733"
 			(at 78.74 43.18 0)
 			(hide yes)
@@
 			)
 		)
-		(property "Value" "BLUE"
+		(property "Value" "GREEN"
 			(at 75.8825 53.34 0)
 			(show_name no)
@@
 			)
 		)
-		(property "Footprint" "LED_SMD:LED_0603_1608Metric"
+		(property "Footprint" "LED_SMD:LED_0805_2012Metric"
 			(at 77.47 57.15 0)
 			(hide yes)
@@
 			)
 		)
-		(property "LCSC Part #" "C965807"
+		(property "LCSC Part #" "C2297"
 			(at 77.47 57.15 0)
 			(hide yes)
@@
 			)
 		)
-		(property "LCSC Part #" "C77009"
+		(property "LCSC Part #" "C52923"
 			(at 133.35 165.1 90)
 			(hide yes)
@@
 			)
 		)
-		(property "LCSC Part #" "C76991"
+		(property "LCSC Part #" "C15525"
 			(at 204.47 64.77 0)
 			(hide yes)
@@
 			)
 		)
-		(property "Footprint" "Button_Switch_SMD:SW_SPST_PTS810"
+		(property "Footprint" "Button_Switch_SMD:SW_SPST_TS-1088-xR025"
 			(at 247.65 88.9 0)
 			(hide yes)
@@
 			)
 		)
-		(property "LCSC Part #" "C221895"
+		(property "LCSC Part #" "C720477"
 			(at 252.73 88.9 90)
 			(hide yes)
@@
 			)
 		)
-		(property "Footprint" "Capacitor_SMD:C_0805_2012Metric"
+		(property "Footprint" "Capacitor_SMD:C_0402_1005Metric"
 			(at 274.0152 140.97 0)
 			(hide yes)
@@
 			)
 		)
-		(property "LCSC Part #" "C5137467"
+		(property "LCSC Part #" "C1525"
 			(at 273.05 137.16 0)
 			(hide yes)
@@
 			)
 		)
-		(property "LCSC Part #" "C2906948"
+		(property "LCSC Part #" "C25905"
 			(at 52.07 128.27 0)
 			(hide yes)
@@
 			)
 		)
-		(property "Footprint" "Resistor_SMD:R_0402_1005Metric"
+		(property "Footprint" "Resistor_SMD:R_0603_1608Metric"
 			(at 258.572 78.74 90)
 			(hide yes)
@@
 			)
 		)
-		(property "LCSC Part #" "C2906861"
+		(property "LCSC Part #" "C25804"
 			(at 260.35 78.74 0)
 			(hide yes)
@@
 			)
 		)
-		(property "Footprint" "Capacitor_SMD:C_0805_2012Metric"
+		(property "Footprint" "Capacitor_SMD:C_0402_1005Metric"
 			(at 244.8052 129.54 0)
 			(hide yes)
@@
 			)
 		)
-		(property "LCSC Part #" "C5137467"
+		(property "LCSC Part #" "C1525"
 			(at 243.84 125.73 90)
 			(hide yes)
@@
 			)
 		)
-		(property "LCSC Part #" "C2906861"
+		(property "LCSC Part #" "C25744"
 			(at 149.86 152.4 90)
 			(hide yes)
@@
 			)
 		)
-		(property "Footprint" "Resistor_SMD:R_0402_1005Metric"
+		(property "Footprint" "Resistor_SMD:R_0603_1608Metric"
 			(at 40.64 71.628 90)
 			(hide yes)
@@
 			)
 		)
-		(property "LCSC Part #" "C2906861"
+		(property "LCSC Part #" "C25804"
 			(at 40.64 69.85 90)
 			(hide yes)
@@
 			)
 		)
-		(property "Footprint" "Button_Switch_SMD:SW_SPST_PTS810"
+		(property "Footprint" "Button_Switch_SMD:SW_SPST_TS-1088-xR025"
 			(at 260.35 138.43 0)
 			(hide yes)
@@
 			)
 		)
-		(property "LCSC Part #" "C221895"
+		(property "LCSC Part #" "C720477"
 			(at 265.43 138.43 90)
 			(hide yes)
@@
 			)
 		)
-		(property "Footprint" "Resistor_SMD:R_0805_2012Metric"
+		(property "Footprint" "Resistor_SMD:R_0402_1005Metric"
 			(at 68.072 147.32 90)
 			(hide yes)
@@
 			)
 		)
-		(property "LCSC Part #" "C2907326"
+		(property "LCSC Part #" "C25900"
 			(at 69.85 147.32 0)
 			(hide yes)
@@
 			)
 		)
-		(property "Footprint" "Diode_SMD:D_SOD-323"
+		(property "Footprint" "Package_TO_SOT_SMD:SOT-23"
 			(at 144.78 156.21 0)
 			(hide yes)
@@
 			)
 		)
-		(property "LCSC Part #" "C5381403"
+		(property "LCSC Part #" "C7502690"
 			(at 144.78 156.21 90)
 			(hide yes)
@@
 			)
 		)
-		(property "Footprint" "Capacitor_SMD:C_0805_2012Metric"
+		(property "Footprint" "Capacitor_SMD:C_0402_1005Metric"
 			(at 157.1752 58.42 0)
 			(hide yes)
@@
 			)
 		)
-		(property "LCSC Part #" "C5137467"
+		(property "LCSC Part #" "C1525"
 			(at 156.21 54.61 0)
 			(hide yes)
@@
 			)
 		)
-		(property "LCSC Part #" "C2909365"
+		(property "LCSC Part #" "C11616"
 			(at 140.97 170.18 90)
 			(hide yes)
@@
 			)
 		)
-		(property "Footprint" "Resistor_SMD:R_0402_1005Metric"
+		(property "Footprint" "Resistor_SMD:R_0603_1608Metric"
 			(at 129.54 51.308 90)
 			(hide yes)
@@
 			)
 		)
-		(property "LCSC Part #" "C42396638"
+		(property "LCSC Part #" "C23147"
 			(at 129.54 49.53 90)
 			(hide yes)
@@
 			)
 		)
-		(property "Footprint" "Capacitor_SMD:C_1210_3225Metric"
+		(property "Footprint" "Capacitor_SMD:C_0603_1608Metric"
 			(at 126.0348 29.21 0)
 			(hide yes)
@@
 			)
 		)
-		(property "LCSC Part #" "C2918511"
+		(property "LCSC Part #" "C59461"
 			(at 127 33.02 0)
 			(hide yes)
@@
 			)
 		)
-		(property "Footprint" "LED_SMD:LED_0603_1608Metric"
+		(property "Footprint" "LED_SMD:LED_0805_2012Metric"
 			(at 77.47 67.31 0)
 			(hide yes)
@@
 			)
 		)
-		(property "LCSC Part #" "C965799"
+		(property "LCSC Part #" "C84256"
 			(at 77.47 67.31 0)
 			(hide yes)
@@
 			)
 		)
-		(property "Footprint" "Capacitor_SMD:C_0805_2012Metric"
+		(property "Footprint" "Capacitor_SMD:C_0402_1005Metric"
 			(at 162.2552 67.31 0)
 			(hide yes)
@@
 			)
 		)
-		(property "LCSC Part #" "C5137467"
+		(property "LCSC Part #" "C1525"
 			(at 161.29 63.5 0)
 			(hide yes)
@@
 			)
 		)
-		(property "LCSC Part #" "C2906948"
+		(property "LCSC Part #" "C25905"
 			(at 55.88 128.27 0)
 			(hide yes)
@@
 			)
 		)
-		(property "Footprint" "Resistor_SMD:R_1206_3216Metric"
+		(property "Footprint" "Resistor_SMD:R_0402_1005Metric"
 			(at 85.09 58.928 90)
 			(hide yes)
@@
 			)
 		)
-		(property "LCSC Part #" "C2907440"
+		(property "LCSC Part #" "C11702"
 			(at 85.09 57.15 90)
 			(hide yes)
@@
 			)
 		)
-		(property "Footprint" "Resistor_SMD:R_0402_1005Metric"
+		(property "Footprint" "Resistor_SMD:R_0603_1608Metric"
 			(at 271.272 128.27 90)
 			(hide yes)
@@
 			)
 		)
-		(property "LCSC Part #" "C2906861"
+		(property "LCSC Part #" "C25804"
 			(at 273.05 128.27 0)
 			(hide yes)
@@
 			)
 		)
-		(property "LCSC Part #" "C76991"
+		(property "LCSC Part #" "C15525"
 			(at 151.13 63.5 0)
 			(hide yes)
@@
 			)
 		)
-		(property "LCSC Part #" "C140177"
+		(property "LCSC Part #" "C25092"
 			(at 160.02 118.11 90)
 			(hide yes)
@@
 			)
 		)
-		(property "LCSC Part #" "C77009"
+		(property "LCSC Part #" "C52923"
 			(at 31.75 38.1 0)
 			(hide yes)
@@
 			)
 		)
-		(property "Value" "GREEN"
+		(property "Value" "YELLOW"
 			(at 141.9225 95.25 0)
 			(show_name no)
@@
 			)
 		)
-		(property "LCSC Part #" "C510026"
+		(property "LCSC Part #" "C89811"
 			(at 143.51 99.06 0)
 			(hide yes)
@@
 			)
 		)
-		(property "LCSC Part #" "C166918"
+		(property "LCSC Part #" "C27592"
 			(at 151.13 99.06 90)
 			(hide yes)
