File: pot_sensor.kicad_sch (KiCad schematic)
At the start: 52 parts, among them J1 USB_C_Receptacle_USB2.0_14P, SW1 EN, SW2 BOOT, U1 ESP32-C3, U2 BQ24074RGT, U3 TPS63900, U4 W25Q80DVSNIG, U5 USBLC6-2P6, U7 HDC3020DEFR, U8 TPS22917DBV, Y1 ABM8-40MHZ

Commit message: Finished and bought
Parts:
- C15, C2: LCSC Part # C52923 -> C14445
- R13: value 10k -> 10K; footprint Resistor_SMD:R_0402_1005Metric -> Resistor_SMD:R_0603_1608Metric; LCSC Part # C25744 -> C25804
Changed lines of the file:
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@@
 			)
 		)
-		(property "LCSC Part #" "C52923"
+		(property "LCSC Part #" "C14445"
 			(at 133.35 165.1 90)
 			(hide yes)
@@
 			)
 		)
-		(property "Value" "10k"
+		(property "Value" "10K"
 			(at 149.86 148.59 90)
 			(show_name no)
@@
 			)
 		)
-		(property "Footprint" "Resistor_SMD:R_0402_1005Metric"
+		(property "Footprint" "Resistor_SMD:R_0603_1608Metric"
 			(at 149.86 154.178 90)
 			(hide yes)
@@
 			)
 		)
-		(property "LCSC Part #" "C25744"
+		(property "LCSC Part #" "C25804"
 			(at 149.86 152.4 90)
 			(hide yes)
@@
 			)
 		)
-		(property "LCSC Part #" "C52923"
+		(property "LCSC Part #" "C14445"
 			(at 31.75 38.1 0)
 			(hide yes)
