File: pot_sensor.kicad_pcb (KiCad board)
At the start: 2 copper layers, 126 x 39.5 mm, 55 parts, among them J1 USB_C_Receptacle_USB2.0_14P, SW1 EN, SW2 BOOT, U1 ESP32-C3, U2 BQ24074RGT, U3 TPS63900, U4 W25Q80DVSNIG, U5 USBLC6-2P6, U7 HDC3020DEFR, U8 TPS22917DBV, Y1 ABM8-40MHZ

Commit message: New pieces
Parts:
- C1, C16, C17, C18, C7, C8, C9: footprint Capacitor_SMD:C_0805_2012Metric -> Capacitor_SMD:C_0402_1005Metric
- C3: footprint Capacitor_SMD:C_1210_3225Metric -> Capacitor_SMD:C_0603_1608Metric
- C5, C6: footprint Capacitor_SMD:C_0603_1608Metric -> Capacitor_SMD:C_0402_1005Metric
- D1: footprint LED_SMD:LED_0603_1608Metric -> LED_SMD:LED_0805_2012Metric
- D2: value BLUE -> GREEN; footprint LED_SMD:LED_0603_1608Metric -> LED_SMD:LED_0805_2012Metric
- D3: value BAT54 -> BAT54A; footprint Diode_SMD:D_SOD-323 -> Package_TO_SOT_SMD:SOT-23
- D4: value GREEN -> YELLOW
- L1: footprint Inductor_SMD:L_1008_2520Metric -> Inductor_SMD:L_0805_2012Metric
- R1, R3: footprint Resistor_SMD:R_1206_3216Metric -> Resistor_SMD:R_0402_1005Metric
- R10, R4, R5, R7: footprint Resistor_SMD:R_0402_1005Metric -> Resistor_SMD:R_0603_1608Metric
- R11, R12: footprint Resistor_SMD:R_0805_2012Metric -> Resistor_SMD:R_0402_1005Metric
- SW1, SW2: footprint Button_Switch_SMD:SW_SPST_PTS810 -> Button_Switch_SMD:SW_SPST_TS-1088-xR025
- moved C7 7.50 mm to (72.0, 55.0), turned to 90 degrees
- moved C9 6.86 mm to (77.0, 56.0)
- moved D3 5.83 mm to (104.5, 76.5), turned to 180 degrees
- moved C6 4.16 mm to (64.7, 68.5)
- moved Y1 3.89 mm to (67.8, 68.1)
- moved C8 3.83 mm to (77.5, 72.0)
- moved C18 3.80 mm to (80.5, 81.5)
- moved C5 3.21 mm to (70.7, 67.5)
- moved C17 2.49 mm to (79.5, 81.5)
- moved R3 1.82 mm to (103.5, 67.5)
- moved SW2 1.64 mm to (81.0, 55.0), turned to 180 degrees
- moved C16 1.56 mm to (78.5, 81.5)
- moved R1 1.53 mm to (102.0, 67.5)
- moved C3 1.28 mm to (94.0, 78.2)
- moved R7 1.17 mm to (73.5, 55.7)
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Connections:
- D3 pad 2: Net-(C12-CIN) -> /ADC_CH4
- JSTconnector1 pad 1: (no net) -> Net-(JSTconnector1-Pad+)
Routing:
- net +3V3: track 45.9 -> 53.8 mm
- net Net-(U1-CHIP_EN): track 140.7 -> 134.7 mm
- net Net-(C6-Pad1): track 10.1 -> 5.68 mm
- net Net-(U1-XTAL_N): track 14.8 -> 11.0 mm
- net Net-(U3-LX1): track 6.82 -> 3.50 mm
- net Net-(U3-LX2): track 6.74 -> 3.50 mm
- net 3V3SPI: track 16.3 -> 19.0 mm, vias 3 -> 2
- net Net-(D1-A): track 4.21 -> 2.00 mm
- net GND: track 46.2 -> 48.1 mm, vias 319 -> 310
- net Net-(U2-EN1): track 11.6 -> 9.87 mm
- net /BOOT_PIN: track 117.2 -> 118.7 mm
- net Net-(D2-A): track 6.48 -> 5.12 mm
- net Net-(U2-ISET): track 3.05 -> 4.11 mm
- net /SDA_line: track 7.29 -> 8.18 mm
- net /SCL_line: track 9.53 -> 10.3 mm
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Other:
- board text added: "POK"
- board text removed: "PGOOD"

Commit message: Broght back labels
Routing:
- net GND: track 48.1 -> 36.5 mm, vias 310 -> 316

Commit message: Finished and bought
Parts:
- D3: value BAT54A -> BAT54
- R13: footprint Resistor_SMD:R_0402_1005Metric -> Resistor_SMD:R_0603_1608Metric
Routing:
- net /1MHz_PWM: track 40.4 -> 39.9 mm
Changed lines of the file:
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@@
 			)
 		)
-		(property "Value" "BAT54A"
+		(property "Value" "BAT54"
 			(at 0 2.4 0)
 			(layer "F.Fab")
@@
 		)
 	)
-	(footprint "Resistor_SMD:R_0402_1005Metric"
+	(footprint "Resistor_SMD:R_0603_1608Metric"
 		(layer "F.Cu")
 		(at 105.5 80.49 -90)
-		(descr "Resistor SMD 0402 (1005 Metric), square (rectangular) end terminal, IPC-7351 nominal, (Body size source: IPC-SM-782 page 72, https://www.pcb-3d.com/wordpress/wp-content/uploads/ipc-sm-782a_amendment_1_and_2.pdf)")
+		(descr "Resistor SMD 0603 (1608 Metric), square (rectangular) end terminal, IPC-7351 nominal, (Body size source: IPC-SM-782 page 72, https://www.pcb-3d.com/wordpress/wp-content/uploads/ipc-sm-782a_amendment_1_and_2.pdf)")
 		(tags "resistor")
 		(property "Reference" "R13"
-			(at 0 0 180)
+			(at 0 0 0)
 			(layer "F.SilkS")
 			(effects
 				(font
-					(size 0.2 0.2)
+					(size 0.3 0.3)
 					(thickness 0.15)
 				)
@@
 		)
 		(property "Value" "10k"
-			(at 0 1.17 90)
+			(at 0 1.43 270)
 			(layer "F.Fab")
 			(effects
@@
 		)
 		(property "Datasheet" ""
-			(at 0 0 90)
+			(at 0 0 270)
 			(layer "F.Fab")
 			(hide yes)
@@
 		)
 		(property "Description" "Resistor"
-			(at 0 0 90)
+			(at 0 0 270)
 			(layer "F.Fab")
 			(hide yes)
@@
 		)
 		(property "KiLib_Generator" "SMD_2terminal_chip_molded"
-			(at 0 0 90)
-			(layer "F.SilkS")
-			(hide yes)
-			(effects
-				(font
-					(size 1 1)
-					(thickness 0.15)
-				)
-			)
-		)
-		(property "PartNumber" "ESR01MZPF1002"
 			(at 0 0 270)
-			(unlocked yes)
-			(layer "F.Fab")
+			(layer "F.SilkS")
 			(hide yes)
 			(effects
@@
 			)
 		)
-		(property "LCSC Part #" "C25744"
+		(property "LCSC Part #" "C25804"
 			(at 0 0 270)
 			(unlocked yes)
@@
 		(duplicate_pad_numbers_are_jumpers no)
 		(fp_line
-			(start -0.153641 0.38)
-			(end 0.153641 0.38)
+			(start -0.237258 0.5225)
+			(end 0.237258 0.5225)
 			(stroke
 				(width 0.12)
@@
 		)
 		(fp_line
-			(start -0.153641 -0.38)
-			(end 0.153641 -0.38)
+			(start -0.237258 -0.5225)
+			(end 0.237258 -0.5225)
 			(stroke
 				(width 0.12)
@@
 		)
 		(fp_rect
-			(start -0.93 -0.47)
-			(end 0.93 0.47)
+			(start -1.48 -0.73)
+			(end 1.48 0.73)
 			(stroke
 				(width 0.05)
@@
 		)
 		(fp_rect
-			(start -0.525 -0.27)
-			(end 0.525 0.27)
+			(start -0.8 -0.4125)
+			(end 0.8 0.4125)
 			(stroke
 				(width 0.1)
@@
 		)
 		(fp_text user "${REFERENCE}"
-			(at 0 0 90)
+			(at 0 0 270)
 			(layer "F.Fab")
 			(effects
 				(font
-					(size 0.26 0.26)
-					(thickness 0.04)
+					(size 0.4 0.4)
+					(thickness 0.06)
 				)
 			)
 		)
 		(pad "1" smd roundrect
-			(at -0.51 0 270)
-			(size 0.54 0.64)
+			(at -0.825 0 270)
+			(size 0.8 0.95)
 			(layers "F.Cu" "F.Mask" "F.Paste")
 			(roundrect_rratio 0.25)
@@
 		)
 		(pad "2" smd roundrect
-			(at 0.51 0 270)
-			(size 0.54 0.64)
+			(at 0.825 0 270)
+			(size 0.8 0.95)
 			(layers "F.Cu" "F.Mask" "F.Paste")
 			(roundrect_rratio 0.25)
@@
 		)
 		(embedded_fonts no)
-		(model "${KICAD10_3DMODEL_DIR}/Resistor_SMD.3dshapes/R_0402_1005Metric.step"
+		(model "${KICAD10_3DMODEL_DIR}/Resistor_SMD.3dshapes/R_0603_1608Metric.step"
 			(offset
 				(xyz 0 0 0)
@@
 	)
 	(segment
-		(start 105.5 79.98)
+		(start 105.185 79.665)
 		(end 103.5625 78.0425)
 		(width 0.25)
@@
 	)
 	(segment
+		(start 105.5 79.665)
+		(end 105.185 79.665)
+		(width 0.25)
+		(layer "F.Cu")
+		(net "Net-(C12-CIN)")
+	)
+	(segment
 		(start 103.5625 76.011592)
 		(end 108.574092 71)
@@
 	)
 	(segment
-		(start 105.5 81.5)
-		(end 105.5 81)
-		(width 0.25)
-		(layer "F.Cu")
-		(net "/1MHz_PWM")
-	)
-	(segment
